File: current_sense/current_sense.kicad_pcb (KiCad board)
At the start: 2 copper layers, 50 x 30 mm, 12 parts, among them J1 Conn_01x02, J2 Conn_01x02, U1 INA213 (50V/V), U2 INA213 (50V/V)

Commit message: Updated silkscreen
Other:
- board text added: "CurrentSense Adapter v1 Copyright 2020 Matthew Lai Licensed under CC BY-SA 4.0 See: https://creativecommons.org/licenses/by-sa/4.0/"
- board text removed: "CurrentSense Adapter v1 Copyright 2020 Matthew Lai Licensed under CC BY-SA 2.0 See: https://creativecommons.org/licenses/by-sa/2.0/"
